File: patient-monitoring-device/electrical/MAX30001.kicad_sch (KiCad schematic)
At the start: 0 parts

Commit message: a few hours later
Parts:
- added C1, C2: 47n, Capacitor_SMD:C_01005_0402Metric, symbol Device:C
- added C13, C14, C17, C18: 10p, Capacitor_SMD:C_01005_0402Metric, symbol Device:C
- added C15: 47p, Capacitor_SMD:C_01005_0402Metric, symbol Device:C
- added C16: 2n, Capacitor_SMD:C_01005_0402Metric, symbol Device:C
- added C3, C4: 1u, Capacitor_SMD:C_01005_0402Metric, symbol Device:C
- added C5, C7: 10u, Capacitor_SMD:C_01005_0402Metric, symbol Device:C
- added C6: 1n, Capacitor_SMD:C_01005_0402Metric, symbol Device:C
- added R1: 324k, Resistor_SMD:R_0201_0603Metric, symbol Device:R_US
- added R2, R3: 200, Resistor_SMD:R_0201_0603Metric, symbol Device:R_US
- added R4, R5: 200k, Resistor_SMD:R_0201_0603Metric, symbol Device:R_US
- added U2: MAX30001, footprints:MAX30001, symbol symbols:MAX30001
Connections:
- new net: C13.1, C15.1, R2.1, U2.A4 (BIP)
- new net: C5.1, U2.C1 (V_{CM})
- new net: C4.1, U2.B6 (CAPP)
- new net: C4.2, U2.B5 (CAPN)
- new net: C6.1, U2.C6 (CPLL)
- new net: C3.1, U2.B1 (V_{BG})
- new net: C1.2, U2.A1 (DRVP)
- new net: C2.2, U2.A2 (DRVN)
- new net: C14.2, C15.2, R3.1, U2.A3 (BIN)
- new net: C16.1, C17.1, R5.1, U2.A5 (ECGP)
- new net: C16.2, C18.2, R4.1, U2.A6 (ECGN)
- new net: R1.1, U2.B2 (R_{BIAS})
- new net: C7.1, U2.D1 (V_{REF})
- new net +1V8: U2.D6 (DVDD), U2.E1 (AVDD)
- new net +2V5: U2.D3 (OVDD)
- new net CSB: U2.E6 (CSB)
- new net FCLK: U2.D5 (FCLK)
- new net GND: C13.2, C14.1, C17.2, C18.1, C3.2, C5.2, C6.2, C7.2, R1.2, U2.B3 (AGND), U2.B4 (AGND), U2.C3 (AGND), U2.C4 (AGND), U2.C5 (DGND), U2.D4 (AGND)
- new net INT2B: U2.E2 (INT2B)
- new net INTB: U2.D2 (INTB)
- new net SCLK: U2.E5 (SCLK)
- new net SDI: U2.E4 (SDI)
- new net SDO: U2.E3 (SDO)
- new net electrode_1/Electrode: C1.1
- new net electrode_2/Electrode: C2.1
- new net electrode_{N}/Electrode: R3.2, R4.2
- new net electrode_{P}/Electrode: R2.2, R5.2
- no-connect marks 0 -> 1
Other:
- added sheet electrode_1 (electrode.kicad_sch)
- added sheet electrode_2 (electrode.kicad_sch)
- added sheet electrode_{N} (electrode.kicad_sch)
- added sheet electrode_{P} (electrode.kicad_sch)
