File: patient-monitoring-device/electrical/MAX86141.kicad_sch (KiCad schematic)
At the start: 0 parts

Commit message: a few hours later
Parts:
- added C10, C11: 10u, Capacitor_SMD:C_01005_0402Metric, symbol Device:C
- added C12: 1u, Capacitor_SMD:C_01005_0402Metric, symbol Device:C
- added C8: C, Capacitor_SMD:C_01005_0402Metric, symbol Device:C
- added C9: 0.1u, Capacitor_SMD:C_01005_0402Metric, symbol Device:C
- added U3: MAX86141, footprints:MAX86141, symbol symbols:MAX86141
Connections:
- new net: C12.2, U3.B5 (VREF)
- new net: C10.1, C9.2
- new net +1V8: C8.1, C9.1, U3.C2 (VDD_{DIG}), U3.D2 (VDD_{ANA})
- new net +5V: C11.2, U3.A1 (V_{LED})
- new net CSB: U3.A5 (CSB)
- new net GND: C10.2, C11.1, C12.1, C8.2, U3.C3 (GND_{DIG}), U3.C4 (GND_{ANA}), U3.D3 (PGND)
- new net INT: U3.B2 (INT)
- new net SCLK: U3.A2 (SCLK)
- new net SDI: U3.A4 (SDI)
- new net SDO: U3.A3 (SDO)
- new net oximeter-sensor/LED1_{DRV}: U3.D1 (LED1_{DRV})
- new net oximeter-sensor/LED2_{DRV}: U3.C1 (LED2_{DRV})
- new net oximeter-sensor/LED3_{DRV}: U3.B1 (LED3_{DRV})
- new net oximeter-sensor/PD1_{IN}: U3.D5 (PD1_{IN})
- new net oximeter-sensor/PD2_{IN}: U3.D4 (PD2_{IN})
- new net oximeter-sensor/PD_{GND}: U3.C5 (PD_{GND})
- no-connect marks 0 -> 2
Other:
- added sheet oximeter-sensor (oximeter-sensor.kicad_sch)
