File: patient-monitoring-device/electrical/patient-monitoring-device.kicad_sch (KiCad schematic)
At the start: 0 parts

Commit message: added max30001 symbool
Other:
- added sheet ESP (ESP02U.kicad_sch)
- added sheet MAX30001 (MAX30001.kicad_sch)
- added sheet MAX86141 (MAX86141.kicad_sch)
Changed lines of the file:
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@@
 	(generator_version "9.0")
 	(paper "A4")
+	(sheet
+		(at 175.26 106.68)
+		(size 39.37 24.13)
+		(exclude_from_sim no)
+		(in_bom yes)
+		(on_board yes)
+		(dnp no)
+		(fields_autoplaced yes)
+		(stroke
+			(width 0.1524)
+			(type solid)
+		)
+		(fill
+			(color 0 0 0 0.0000)
+		)
+		(property "Sheetname" "MAX30001"
+			(at 175.26 105.9684 0)
+			(effects
+				(font
+					(size 1.27 1.27)
+				)
+				(justify left bottom)
+			)
+		)
+		(property "Sheetfile" "MAX30001.kicad_sch"
+			(at 175.26 131.3946 0)
+			(effects
+				(font
+					(size 1.27 1.27)
+				)
+				(justify left top)
+			)
+		)
+		(instances
+			(project "patient-monitoring-device"
+				(path "/c785af1e-244f-4b75-a94e-a052bfe737f0"
+					(page "4")
+				)
+			)
+		)
+	)
+	(sheet
+		(at 102.87 50.8)
+		(size 29.21 35.56)
+		(exclude_from_sim no)
+		(in_bom yes)
+		(on_board yes)
+		(dnp no)
+		(fields_autoplaced yes)
+		(stroke
+			(width 0.1524)
+			(type solid)
+		)
+		(fill
+			(color 0 0 0 0.0000)
+		)
+		(property "Sheetname" "ESP"
+			(at 102.87 50.0884 0)
+			(effects
+				(font
+					(size 1.27 1.27)
+				)
+				(justify left bottom)
+			)
+		)
+		(property "Sheetfile" "ESP02U.kicad_sch"
+			(at 102.87 86.9446 0)
+			(effects
+				(font
+					(size 1.27 1.27)
+				)
+				(justify left top)
+			)
+		)
+		(instances
+			(project "patient-monitoring-device"
+				(path "/c785af1e-244f-4b75-a94e-a052bfe737f0"
+					(page "2")
+				)
+			)
+		)
+	)
+	(sheet
+		(at 184.15 53.34)
+		(size 45.72 36.83)
+		(exclude_from_sim no)
+		(in_bom yes)
+		(on_board yes)
+		(dnp no)
+		(fields_autoplaced yes)
+		(stroke
+			(width 0.1524)
+			(type solid)
+		)
+		(fill
+			(color 0 0 0 0.0000)
+		)
+		(property "Sheetname" "MAX86141"
+			(at 184.15 52.6284 0)
+			(effects
+				(font
+					(size 1.27 1.27)
+				)
+				(justify left bottom)
+			)
+		)
+		(property "Sheetfile" "MAX86141.kicad_sch"
+			(at 184.15 90.7546 0)
+			(effects
+				(font
+					(size 1.27 1.27)
+				)
+				(justify left top)
+			)
+		)
+		(instances
+			(project "patient-monitoring-device"
+				(path "/c785af1e-244f-4b75-a94e-a052bfe737f0"
+					(page "3")
+				)
+			)
+		)
+	)
 	(sheet_instances
 		(path "/"

Commit message: a few hours later
Other:
- added sheet power (power.kicad_sch)
- sheet ESP ports: added CS_{ECG,R}, CS_{SpO2}, FCK, INT_{B2}, INT_{B}, INT_{SpO2}, MISO, MOSI, SCK; removed none
- sheet MAX30001 ports: added CSB, FCLK, INT2B, INTB, SCLK, SDI, SDO; removed none
- sheet MAX86141 ports: added CSB, INT, SCLK, SDI, SDO; removed none
